Commit message: Add Models

File: urdf/peg_round.urdf (robot description, URDF)
Before this commit: robot hole_round, 1 links, 0 joints
Links:
- removed link hole_link
- added link peg_link, mass 0.1; collision mesh filename=meshes/peg/peg_round.STL scale=0.001 0.001 0.001; visual mesh filename=meshes/peg/peg_round.STL scale=0.001 0.001 0.001
