Commit message: Romove build add tool changing methods

File: urdf/hole_round.urdf (robot description, URDF)
Before this commit: robot peg_round, 1 links, 0 joints
Links:
- removed link peg_link
- added link hole_link, mass 0.1; collision mesh filename=meshes/hole/hole_round.STL scale=0.001 0.001 0.001; visual mesh filename=meshes/hole/hole_round.STL scale=0.001 0.001 0.001
