Commit message: Add camera

File: tests/urdf/ur5e_pybullet.urdf (robot description, URDF)
Before this commit: robot ur5e, 12 links, 11 joints
Links:
- added link camera_link, mass 0
Joints:
- added joint camera_link_joint: type fixed, parent tool0, child camera_link, origin xyz= 0.00 -0.00 0.1 rpy=0.0 0 0.0

Commit message: Fix fov

File: tests/urdf/ur5e_pybullet.urdf (robot description, URDF)
Before this commit: robot ur5e, 13 links, 12 joints
Joints:
- joint camera_link_joint: origin xyz= 0.00 -0.00 0.1 rpy=0.0 0 0.0 -> xyz= 0.00 -0.00 0.1 rpy=-0.2 0 0.0

Commit message: Fix reset_ee_state for non default frame, fix jacobian calculation for also non default (now 'global') frame

File: tests/urdf/ur5e_pybullet.urdf (robot description, URDF)
Before this commit: robot ur5e, 13 links, 12 joints
Links:
- removed link world
- added link bworld
Joints:
- joint world_joint: parent world -> bworld
